File: BufferPortB.sch (KiCad schematic (older format))
At the start: 4 parts, among them U61 74ABT574, U62 74ABT574

Commit message: Update broken footprints for resistors and capacitors.
Parts:
- C61, C62: footprint Capacitor_SMD:C_0603_1608Metric_Pad1.05x0.95mm_HandSolder -> Capacitor_SMD:C_0201_0603Metric_Pad0.64x0.40mm_HandSolder
Changed lines of the file:
@@
 F 0 "C61" H 1215 7196 50  0000 L CNN
 F 1 "100nF" H 1215 7105 50  0000 L CNN
-F 2 "Capacitor_SMD:C_0603_1608Metric_Pad1.05x0.95mm_HandSolder" H 1138 7000 50  0001 C CNN
+F 2 "Capacitor_SMD:C_0201_0603Metric_Pad0.64x0.40mm_HandSolder" H 1138 7000 50  0001 C CNN
 F 3 "~" H 1100 7150 50  0001 C CNN
 	1    1100 7150
@@
 F 0 "C62" H 1665 7196 50  0000 L CNN
 F 1 "100nF" H 1665 7105 50  0000 L CNN
-F 2 "Capacitor_SMD:C_0603_1608Metric_Pad1.05x0.95mm_HandSolder" H 1588 7000 50  0001 C CNN
+F 2 "Capacitor_SMD:C_0201_0603Metric_Pad0.64x0.40mm_HandSolder" H 1588 7000 50  0001 C CNN
 F 3 "~" H 1550 7150 50  0001 C CNN
 	1    1550 7150

Commit message: Fix typo in ID
Parts:
- C61, C62: footprint Capacitor_SMD:C_0201_0603Metric_Pad0.64x0.40mm_HandSolder -> Capacitor_SMD:C_0603_1608Metric_Pad1.08x0.95mm_HandSolder
Changed lines of the file:
@@
 F 0 "C61" H 1215 7196 50  0000 L CNN
 F 1 "100nF" H 1215 7105 50  0000 L CNN
-F 2 "Capacitor_SMD:C_0201_0603Metric_Pad0.64x0.40mm_HandSolder" H 1138 7000 50  0001 C CNN
+F 2 "Capacitor_SMD:C_0603_1608Metric_Pad1.08x0.95mm_HandSolder" H 1138 7000 50  0001 C CNN
 F 3 "~" H 1100 7150 50  0001 C CNN
 	1    1100 7150
@@
 F 0 "C62" H 1665 7196 50  0000 L CNN
 F 1 "100nF" H 1665 7105 50  0000 L CNN
-F 2 "Capacitor_SMD:C_0201_0603Metric_Pad0.64x0.40mm_HandSolder" H 1588 7000 50  0001 C CNN
+F 2 "Capacitor_SMD:C_0603_1608Metric_Pad1.08x0.95mm_HandSolder" H 1588 7000 50  0001 C CNN
 F 3 "~" H 1550 7150 50  0001 C CNN
 	1    1550 7150

Commit message: Checkpoint while routing PCB.
A lot of parts have been placed and about a quarter of the board is routed.
Parts:
- renumbered U61 to U60, U62 to U61
Changed lines of the file:
@@
 AR Path="/5FF41DF6/5FC5F3B1/5FDD26FD" Ref="#PWR?"  Part="1"
 AR Path="/60B264DC/5FCD7CF6/5FDD26FD" Ref="#PWR?"  Part="1"
-AR Path="/60906BCD/5FDCBC44/5FDD26FD" Ref="#PWR0369"  Part="1"
-F 0 "#PWR0369" H 5150 2850 50  0001 C CNN
+AR Path="/60906BCD/5FDCBC44/5FDD26FD" Ref="#PWR0365"  Part="1"
+F 0 "#PWR0365" H 5150 2850 50  0001 C CNN
 F 1 "GND" V 5155 2972 50  0000 R CNN
 F 2 "" H 5150 3100 50  0001 C CNN
@@
 AR Path="/5FF41DF6/5FC5F3B1/5FDD271D" Ref="#PWR?"  Part="1"
 AR Path="/60B264DC/5FCD7CF6/5FDD271D" Ref="#PWR?"  Part="1"
-AR Path="/60906BCD/5FDCBC44/5FDD271D" Ref="#PWR0372"  Part="1"
-F 0 "#PWR0372" H 5650 3150 50  0001 C CNN
+AR Path="/60906BCD/5FDCBC44/5FDD271D" Ref="#PWR0368"  Part="1"
+F 0 "#PWR0368" H 5650 3150 50  0001 C CNN
 F 1 "GND" H 5655 3227 50  0000 C CNN
 F 2 "" H 5650 3400 50  0001 C CNN
@@
 AR Path="/5FF41DF6/5FC5F3B1/5FDD2723" Ref="#PWR?"  Part="1"
 AR Path="/60B264DC/5FCD7CF6/5FDD2723" Ref="#PWR?"  Part="1"
-AR Path="/60906BCD/5FDCBC44/5FDD2723" Ref="#PWR0371"  Part="1"
-F 0 "#PWR0371" H 5650 1650 50  0001 C CNN
+AR Path="/60906BCD/5FDCBC44/5FDD2723" Ref="#PWR0367"  Part="1"
+F 0 "#PWR0367" H 5650 1650 50  0001 C CNN
 F 1 "VCC" H 5667 1973 50  0000 C CNN
 F 2 "" H 5650 1800 50  0001 C CNN
@@
 AR Path="/5FF41DF6/5FC5F3B1/5FDD2743" Ref="U?"  Part="1"
 AR Path="/60B264DC/5FCD7CF6/5FDD2743" Ref="U?"  Part="1"
-AR Path="/60906BCD/5FDCBC44/5FDD2743" Ref="U61"  Part="1"
-F 0 "U61" H 5400 3400 50  0000 C CNN
+AR Path="/60906BCD/5FDCBC44/5FDD2743" Ref="U60"  Part="1"
+F 0 "U60" H 5400 3400 50  0000 C CNN
 F 1 "74ABT574" H 5400 3300 50  0000 C CNN
 F 2 "Package_SO:TSSOP-20_4.4x6.5mm_P0.65mm" H 5650 2600 50  0001 C CNN
@@
 AR Path="/5FF41DF6/5FC5F3B1/5FDD274F" Ref="#PWR?"  Part="1"
 AR Path="/60B264DC/5FCD7CF6/5FDD274F" Ref="#PWR?"  Part="1"
-AR Path="/60906BCD/5FDCBC44/5FDD274F" Ref="#PWR0365"  Part="1"
-F 0 "#PWR0365" H 1100 6850 50  0001 C CNN
+AR Path="/60906BCD/5FDCBC44/5FDD274F" Ref="#PWR0361"  Part="1"
+F 0 "#PWR0361" H 1100 6850 50  0001 C CNN
 F 1 "VCC" H 1117 7173 50  0000 C CNN
 F 2 "" H 1100 7000 50  0001 C CNN
@@
 AR Path="/5FF41DF6/5FC5F3B1/5FDD2755" Ref="#PWR?"  Part="1"
 AR Path="/60B264DC/5FCD7CF6/5FDD2755" Ref="#PWR?"  Part="1"
-AR Path="/60906BCD/5FDCBC44/5FDD2755" Ref="#PWR0366"  Part="1"
-F 0 "#PWR0366" H 1100 7150 50  0001 C CNN
+AR Path="/60906BCD/5FDCBC44/5FDD2755" Ref="#PWR0362"  Part="1"
+F 0 "#PWR0362" H 1100 7150 50  0001 C CNN
 F 1 "GND" H 1105 7227 50  0000 C CNN
 F 2 "" H 1100 7400 50  0001 C CNN
@@
 AR Path="/5FF41DF6/5FC5F3B1/5FDD2762" Ref="#PWR?"  Part="1"
 AR Path="/60B264DC/5FCD7CF6/5FDD2762" Ref="#PWR?"  Part="1"
-AR Path="/60906BCD/5FDCBC44/5FDD2762" Ref="#PWR0367"  Part="1"
-F 0 "#PWR0367" H 1550 6850 50  0001 C CNN
+AR Path="/60906BCD/5FDCBC44/5FDD2762" Ref="#PWR0363"  Part="1"
+F 0 "#PWR0363" H 1550 6850 50  0001 C CNN
 F 1 "VCC" H 1567 7173 50  0000 C CNN
 F 2 "" H 1550 7000 50  0001 C CNN
@@
 AR Path="/5FF41DF6/5FC5F3B1/5FDD2768" Ref="#PWR?"  Part="1"
 AR Path="/60B264DC/5FCD7CF6/5FDD2768" Ref="#PWR?"  Part="1"
-AR Path="/60906BCD/5FDCBC44/5FDD2768" Ref="#PWR0368"  Part="1"
-F 0 "#PWR0368" H 1550 7150 50  0001 C CNN
+AR Path="/60906BCD/5FDCBC44/5FDD2768" Ref="#PWR0364"  Part="1"
+F 0 "#PWR0364" H 1550 7150 50  0001 C CNN
 F 1 "GND" H 1555 7227 50  0000 C CNN
 F 2 "" H 1550 7400 50  0001 C CNN
@@
 AR Path="/5FF41DF6/5FC5F3B1/5FDD2770" Ref="#PWR?"  Part="1"
 AR Path="/60B264DC/5FCD7CF6/5FDD2770" Ref="#PWR?"  Part="1"
-AR Path="/60906BCD/5FDCBC44/5FDD2770" Ref="#PWR0370"  Part="1"
-F 0 "#PWR0370" H 5150 4900 50  0001 C CNN
+AR Path="/60906BCD/5FDCBC44/5FDD2770" Ref="#PWR0366"  Part="1"
+F 0 "#PWR0366" H 5150 4900 50  0001 C CNN
 F 1 "GND" V 5155 5022 50  0000 R CNN
 F 2 "" H 5150 5150 50  0001 C CNN
@@
 AR Path="/5FF41DF6/5FC5F3B1/5FDD278F" Ref="#PWR?"  Part="1"
 AR Path="/60B264DC/5FCD7CF6/5FDD278F" Ref="#PWR?"  Part="1"
-AR Path="/60906BCD/5FDCBC44/5FDD278F" Ref="#PWR0374"  Part="1"
-F 0 "#PWR0374" H 5650 5200 50  0001 C CNN
+AR Path="/60906BCD/5FDCBC44/5FDD278F" Ref="#PWR0370"  Part="1"
+F 0 "#PWR0370" H 5650 5200 50  0001 C CNN
 F 1 "GND" H 5655 5277 50  0000 C CNN
 F 2 "" H 5650 5450 50  0001 C CNN
@@
 AR Path="/5FF41DF6/5FC5F3B1/5FDD2795" Ref="#PWR?"  Part="1"
 AR Path="/60B264DC/5FCD7CF6/5FDD2795" Ref="#PWR?"  Part="1"
-AR Path="/60906BCD/5FDCBC44/5FDD2795" Ref="#PWR0373"  Part="1"
-F 0 "#PWR0373" H 5650 3700 50  0001 C CNN
+AR Path="/60906BCD/5FDCBC44/5FDD2795" Ref="#PWR0369"  Part="1"
+F 0 "#PWR0369" H 5650 3700 50  0001 C CNN
 F 1 "VCC" H 5667 4023 50  0000 C CNN
 F 2 "" H 5650 3850 50  0001 C CNN
@@
 AR Path="/5FF41DF6/5FC5F3B1/5FDD27B3" Ref="U?"  Part="1"
 AR Path="/60B264DC/5FCD7CF6/5FDD27B3" Ref="U?"  Part="1"
-AR Path="/60906BCD/5FDCBC44/5FDD27B3" Ref="U62"  Part="1"
-F 0 "U62" H 5400 5450 50  0000 C CNN
+AR Path="/60906BCD/5FDCBC44/5FDD27B3" Ref="U61"  Part="1"
+F 0 "U61" H 5400 5450 50  0000 C CNN
 F 1 "74ABT574" H 5400 5350 50  0000 C CNN
 F 2 "Package_SO:TSSOP-20_4.4x6.5mm_P0.65mm" H 5650 4650 50  0001 C CNN

Commit message: checkpoint
Connections:
- net D0 renamed Bin0
- net D1 renamed Bin1
- net D10 renamed Bin10
- net D11 renamed Bin11
- net D12 renamed Bin12
- net D13 renamed Bin13
- net D14 renamed Bin14
- net D15 renamed Bin15
- net D2 renamed Bin2
- net D3 renamed Bin3
- net D4 renamed Bin4
- net D5 renamed Bin5
- net D6 renamed Bin6
- net D7 renamed Bin7
- net D8 renamed Bin8
- net D9 renamed Bin9
- net Q0 renamed Bout0
- net Q1 renamed Bout1
- net Q10 renamed Bout10
- net Q11 renamed Bout11
- net Q12 renamed Bout12
- net Q13 renamed Bout13
- net Q14 renamed Bout14
- net Q15 renamed Bout15
- net Q2 renamed Bout2
- net Q3 renamed Bout3
- net Q4 renamed Bout4
- net Q5 renamed Bout5
- net Q6 renamed Bout6
- net Q7 renamed Bout7
- net Q8 renamed Bout8
- net Q9 renamed Bout9
Changed lines of the file:
@@
 	5000 3000 5150 3000
 Text Label 4950 2800 2    50   ~ 0
-D7
+Bin7
 Wire Wire Line
 	4750 2800 5150 2800
@@
 	4650 2700 4750 2800
 Text Label 4950 2700 2    50   ~ 0
-D6
+Bin6
 Wire Wire Line
 	4750 2700 5150 2700
@@
 	4650 2600 4750 2700
 Text Label 4950 2600 2    50   ~ 0
-D5
+Bin5
 Wire Wire Line
 	4750 2600 5150 2600
@@
 	4650 2500 4750 2600
 Text Label 4950 2500 2    50   ~ 0
-D4
+Bin4
 Wire Wire Line
 	4750 2500 5150 2500
@@
 	4650 2400 4750 2500
 Text Label 4950 2400 2    50   ~ 0
-D3
+Bin3
 Wire Wire Line
 	4750 2400 5150 2400
@@
 	4650 2300 4750 2400
 Text Label 4950 2300 2    50   ~ 0
-D2
+Bin2
 Wire Wire Line
 	4750 2300 5150 2300
@@
 	4650 2200 4750 2300
 Text Label 4950 2200 2    50   ~ 0
-D1
+Bin1
 Wire Wire Line
 	4750 2200 5150 2200
@@
 	4650 2100 4750 2200
 Text Label 4950 2100 2    50   ~ 0
-D0
+Bin0
 Wire Wire Line
 	4750 2100 5150 2100
@@
 $EndComp
 Text HLabel 3800 1850 0    50   Input ~ 0
-D[0..15]
+Bin[0..15]
 Text Label 6350 2800 0    50   ~ 0
-Q7
+Bout7
 Wire Wire Line
 	6550 2800 6150 2800
@@
 	6650 2700 6550 2800
 Text Label 6350 2700 0    50   ~ 0
-Q6
+Bout6
 Wire Wire Line
 	6550 2700 6150 2700
@@
 	6650 2600 6550 2700
 Text Label 6350 2600 0    50   ~ 0
-Q5
+Bout5
 Wire Wire Line
 	6550 2600 6150 2600
@@
 	6650 2500 6550 2600
 Text Label 6350 2500 0    50   ~ 0
-Q4
+Bout4
 Wire Wire Line
 	6550 2500 6150 2500
@@
 	6650 2400 6550 2500
 Text Label 6350 2400 0    50   ~ 0
-Q3
+Bout3
 Wire Wire Line
 	6550 2400 6150 2400
@@
 	6650 2300 6550 2400
 Text Label 6350 2300 0    50   ~ 0
-Q2
+Bout2
 Wire Wire Line
 	6550 2300 6150 2300
@@
 	6650 2200 6550 2300
 Text Label 6350 2200 0    50   ~ 0
-Q1
+Bout1
 Wire Wire Line
 	6550 2200 6150 2200
@@
 	6650 2100 6550 2200
 Text Label 6350 2100 0    50   ~ 0
-Q0
+Bout0
 Wire Wire Line
 	6550 2100 6150 2100
@@
 	5000 5050 5150 5050
 Text Label 4950 4850 2    50   ~ 0
-D15
+Bin15
 Wire Wire Line
 	4750 4850 5150 4850
@@
 	4650 4750 4750 4850
 Text Label 4950 4750 2    50   ~ 0
-D14
+Bin14
 Wire Wire Line
 	4750 4750 5150 4750
@@
 	4650 4650 4750 4750
 Text Label 4950 4650 2    50   ~ 0
-D13
+Bin13
 Wire Wire Line
 	4750 4650 5150 4650
@@
 	4650 4550 4750 4650
 Text Label 4950 4550 2    50   ~ 0
-D12
+Bin12
 Wire Wire Line
 	4750 4550 5150 4550
@@
 	4650 4450 4750 4550
 Text Label 4950 4450 2    50   ~ 0
-D11
+Bin11
 Wire Wire Line
 	4750 4450 5150 4450
@@
 	4650 4350 4750 4450
 Text Label 4950 4350 2    50   ~ 0
-D10
+Bin10
 Wire Wire Line
 	4750 4350 5150 4350
@@
 	4650 4250 4750 4350
 Text Label 4950 4250 2    50   ~ 0
-D9
+Bin9
 Wire Wire Line
 	4750 4250 5150 4250
@@
 	4650 4150 4750 4250
 Text Label 4950 4150 2    50   ~ 0
-D8
+Bin8
 Wire Wire Line
 	4750 4150 5150 4150
@@
 $EndComp
 Text Label 6350 4850 0    50   ~ 0
-Q15
+Bout15
 Wire Wire Line
 	6550 4850 6150 4850
@@
 	6650 4750 6550 4850
 Text Label 6350 4750 0    50   ~ 0
-Q14
+Bout14
 Wire Wire Line
 	6550 4750 6150 4750
@@
 	6650 4650 6550 4750
 Text Label 6350 4650 0    50   ~ 0
-Q13
+Bout13
 Wire Wire Line
 	6550 4650 6150 4650
@@
 	6650 4550 6550 4650
 Text Label 6350 4550 0    50   ~ 0
-Q12
+Bout12
 Wire Wire Line
 	6550 4550 6150 4550
@@
 	6650 4450 6550 4550
 Text Label 6350 4450 0    50   ~ 0
-Q11
+Bout11
 Wire Wire Line
 	6550 4450 6150 4450
@@
 	6650 4350 6550 4450
 Text Label 6350 4350 0    50   ~ 0
-Q10
+Bout10
 Wire Wire Line
 	6550 4350 6150 4350
@@
 	6650 4250 6550 4350
 Text Label 6350 4250 0    50   ~ 0
-Q9
+Bout9
 Wire Wire Line
 	6550 4250 6150 4250
@@
 	6650 4150 6550 4250
 Text Label 6350 4150 0    50   ~ 0
-Q8
+Bout8
 Wire Wire Line
 	6550 4150 6150 4150
@@
 $EndComp
 Text HLabel 7500 1800 2    50   Output ~ 0
-Q[0..15]
+Bout[0..15]
 Wire Bus Line
 	4650 1850 4650 4750
