File: REG_EX.sch (KiCad schematic (older format))
At the start: 2 parts, among them U30 74AHCT04

Commit message: Update broken footprints for resistors and capacitors.
Parts:
- C31: footprint Capacitor_SMD:C_0603_1608Metric_Pad1.05x0.95mm_HandSolder -> Capacitor_SMD:C_0201_0603Metric_Pad0.64x0.40mm_HandSolder
Changed lines of the file:
@@
 F 0 "C31" H 965 7246 50  0000 L CNN
 F 1 "100nF" H 965 7155 50  0000 L CNN
-F 2 "Capacitor_SMD:C_0603_1608Metric_Pad1.05x0.95mm_HandSolder" H 888 7050 50  0001 C CNN
+F 2 "Capacitor_SMD:C_0201_0603Metric_Pad0.64x0.40mm_HandSolder" H 888 7050 50  0001 C CNN
 F 3 "~" H 850 7200 50  0001 C CNN
 	1    850  7200

Commit message: Fix typo in ID
Parts:
- C31: footprint Capacitor_SMD:C_0201_0603Metric_Pad0.64x0.40mm_HandSolder -> Capacitor_SMD:C_0603_1608Metric_Pad1.08x0.95mm_HandSolder
Changed lines of the file:
@@
 F 0 "C31" H 965 7246 50  0000 L CNN
 F 1 "100nF" H 965 7155 50  0000 L CNN
-F 2 "Capacitor_SMD:C_0201_0603Metric_Pad0.64x0.40mm_HandSolder" H 888 7050 50  0001 C CNN
+F 2 "Capacitor_SMD:C_0603_1608Metric_Pad1.08x0.95mm_HandSolder" H 888 7050 50  0001 C CNN
 F 3 "~" H 850 7200 50  0001 C CNN
 	1    850  7200

Commit message: Update component footprints.
I'll use TSSOP footprints for all logic chips that I can. (checking against
Mouser online) I soldered a TSSOP for the sound card and it wasn't bad.
I think I can manage this and save some additional board space.
Parts:
- U30: footprint Package_SO:SOIC-14_3.9x8.7mm_P1.27mm -> Package_SO:TSSOP-14_4.4x5mm_P0.65mm
Changed lines of the file:
@@
 F 0 "U30" H -850 5900 50  0000 C CNN
 F 1 "74AHCT04" H -850 5800 50  0000 C CNN
-F 2 "Package_SO:SOIC-14_3.9x8.7mm_P1.27mm" H -850 5850 50  0001 C CNN
+F 2 "Package_SO:TSSOP-14_4.4x5mm_P0.65mm" H -850 5850 50  0001 C CNN
 F 3 "http://www.ti.com/general/docs/suppproductinfo.tsp?distId=26&gotoUrl=http%3A%2F%2Fwww.ti.com%2Flit%2Fgpn%2Fsn74ahct04" H -850 5850 50  0001 C CNN
 	7    -850 5850
@@
 F 0 "U30" H -550 5367 50  0000 C CNN
 F 1 "74AHCT04" H -550 5276 50  0000 C CNN
-F 2 "Package_SO:SOIC-14_3.9x8.7mm_P1.27mm" H -550 5050 50  0001 C CNN
+F 2 "Package_SO:TSSOP-14_4.4x5mm_P0.65mm" H -550 5050 50  0001 C CNN
 F 3 "http://www.ti.com/general/docs/suppproductinfo.tsp?distId=26&gotoUrl=http%3A%2F%2Fwww.ti.com%2Flit%2Fgpn%2Fsn74ahct04" H -550 5050 50  0001 C CNN
 	6    -550 5050
@@
 F 0 "U30" H -550 3367 50  0000 C CNN
 F 1 "74AHCT04" H -550 3276 50  0000 C CNN
-F 2 "Package_SO:SOIC-14_3.9x8.7mm_P1.27mm" H -550 3050 50  0001 C CNN
+F 2 "Package_SO:TSSOP-14_4.4x5mm_P0.65mm" H -550 3050 50  0001 C CNN
 F 3 "http://www.ti.com/general/docs/suppproductinfo.tsp?distId=26&gotoUrl=http%3A%2F%2Fwww.ti.com%2Flit%2Fgpn%2Fsn74ahct04" H -550 3050 50  0001 C CNN
 	2    -550 3050
@@
 F 0 "U30" H -550 4867 50  0000 C CNN
 F 1 "74AHCT04" H -550 4776 50  0000 C CNN
-F 2 "Package_SO:SOIC-14_3.9x8.7mm_P1.27mm" H -550 4550 50  0001 C CNN
+F 2 "Package_SO:TSSOP-14_4.4x5mm_P0.65mm" H -550 4550 50  0001 C CNN
 F 3 "http://www.ti.com/general/docs/suppproductinfo.tsp?distId=26&gotoUrl=http%3A%2F%2Fwww.ti.com%2Flit%2Fgpn%2Fsn74ahct04" H -550 4550 50  0001 C CNN
 	5    -550 4550
@@
 F 0 "U30" H -550 4367 50  0000 C CNN
 F 1 "74AHCT04" H -550 4276 50  0000 C CNN
-F 2 "Package_SO:SOIC-14_3.9x8.7mm_P1.27mm" H -550 4050 50  0001 C CNN
+F 2 "Package_SO:TSSOP-14_4.4x5mm_P0.65mm" H -550 4050 50  0001 C CNN
 F 3 "http://www.ti.com/general/docs/suppproductinfo.tsp?distId=26&gotoUrl=http%3A%2F%2Fwww.ti.com%2Flit%2Fgpn%2Fsn74ahct04" H -550 4050 50  0001 C CNN
 	4    -550 4050
@@
 F 0 "U30" H -550 3867 50  0000 C CNN
 F 1 "74AHCT04" H -550 3776 50  0000 C CNN
-F 2 "Package_SO:SOIC-14_3.9x8.7mm_P1.27mm" H -550 3550 50  0001 C CNN
+F 2 "Package_SO:TSSOP-14_4.4x5mm_P0.65mm" H -550 3550 50  0001 C CNN
 F 3 "http://www.ti.com/general/docs/suppproductinfo.tsp?distId=26&gotoUrl=http%3A%2F%2Fwww.ti.com%2Flit%2Fgpn%2Fsn74ahct04" H -550 3550 50  0001 C CNN
 	3    -550 3550
@@
 F 0 "U30" H 4650 2467 50  0000 C CNN
 F 1 "74AHCT04" H 4650 2376 50  0000 C CNN
-F 2 "Package_SO:SOIC-14_3.9x8.7mm_P1.27mm" H 4650 2150 50  0001 C CNN
+F 2 "Package_SO:TSSOP-14_4.4x5mm_P0.65mm" H 4650 2150 50  0001 C CNN
 F 3 "http://www.ti.com/general/docs/suppproductinfo.tsp?distId=26&gotoUrl=http%3A%2F%2Fwww.ti.com%2Flit%2Fgpn%2Fsn74ahct04" H 4650 2150 50  0001 C CNN
 	1    4650 2150

Commit message: Checkpoint while routing PCB.
A lot of parts have been placed and about a quarter of the board is routed.
Parts:
- removed unit 2 of U30
- renumbered U30 to U29
Connections:
- wire segments 19 -> 18
- no-connect marks 5 -> 4
Changed lines of the file:
@@
 Wire Bus Line
 	6700 4250 6350 4250
-NoConn ~ -250 3050
 NoConn ~ -250 4550
 NoConn ~ -250 5050
@@
 AR Path="/5D2C0720/5FC492C0" Ref="U?"  Part="7"
 AR Path="/5D2C07CD/5FC492C0" Ref="U?"  Part="7"
-AR Path="/60A72859/5FC492C0" Ref="U30"  Part="7"
-F 0 "U30" H -850 5900 50  0000 C CNN
+AR Path="/60A72859/5FC492C0" Ref="U29"  Part="7"
+F 0 "U29" H -850 5900 50  0000 C CNN
 F 1 "74AHCT04" H -850 5800 50  0000 C CNN
 F 2 "Package_SO:TSSOP-14_4.4x5mm_P0.65mm" H -850 5850 50  0001 C CNN
@@
 AR Path="/5D2C0720/5FC492C6" Ref="U?"  Part="6"
 AR Path="/5D2C07CD/5FC492C6" Ref="U?"  Part="6"
-AR Path="/60A72859/5FC492C6" Ref="U30"  Part="6"
-F 0 "U30" H -550 5367 50  0000 C CNN
+AR Path="/60A72859/5FC492C6" Ref="U29"  Part="6"
+F 0 "U29" H -550 5367 50  0000 C CNN
 F 1 "74AHCT04" H -550 5276 50  0000 C CNN
 F 2 "Package_SO:TSSOP-14_4.4x5mm_P0.65mm" H -550 5050 50  0001 C CNN
 F 3 "http://www.ti.com/general/docs/suppproductinfo.tsp?distId=26&gotoUrl=http%3A%2F%2Fwww.ti.com%2Flit%2Fgpn%2Fsn74ahct04" H -550 5050 50  0001 C CNN
 	6    -550 5050
-	1    0    0    -1
-$EndComp
-$Comp
-L 74xx:74LS04 U?
-U 2 1 5FC492CC
-P -550 3050
-AR Path="/5D8005AF/5D800744/5FC492CC" Ref="U?"  Part="6"
-AR Path="/5D2C0720/5FC492CC" Ref="U?"  Part="2"
-AR Path="/5D2C07CD/5FC492CC" Ref="U?"  Part="2"
-AR Path="/60A72859/5FC492CC" Ref="U30"  Part="2"
-F 0 "U30" H -550 3367 50  0000 C CNN
-F 1 "74AHCT04" H -550 3276 50  0000 C CNN
-F 2 "Package_SO:TSSOP-14_4.4x5mm_P0.65mm" H -550 3050 50  0001 C CNN
-F 3 "http://www.ti.com/general/docs/suppproductinfo.tsp?distId=26&gotoUrl=http%3A%2F%2Fwww.ti.com%2Flit%2Fgpn%2Fsn74ahct04" H -550 3050 50  0001 C CNN
-	2    -550 3050
 	1    0    0    -1
 $EndComp
@@
 AR Path="/5D2C0720/5FC492D2" Ref="U?"  Part="5"
 AR Path="/5D2C07CD/5FC492D2" Ref="U?"  Part="5"
-AR Path="/60A72859/5FC492D2" Ref="U30"  Part="5"
-F 0 "U30" H -550 4867 50  0000 C CNN
+AR Path="/60A72859/5FC492D2" Ref="U29"  Part="5"
+F 0 "U29" H -550 4867 50  0000 C CNN
 F 1 "74AHCT04" H -550 4776 50  0000 C CNN
 F 2 "Package_SO:TSSOP-14_4.4x5mm_P0.65mm" H -550 4550 50  0001 C CNN
@@
 AR Path="/5D2C0720/5FC492D8" Ref="U?"  Part="4"
 AR Path="/5D2C07CD/5FC492D8" Ref="U?"  Part="4"
-AR Path="/60A72859/5FC492D8" Ref="U30"  Part="4"
-F 0 "U30" H -550 4367 50  0000 C CNN
+AR Path="/60A72859/5FC492D8" Ref="U29"  Part="4"
+F 0 "U29" H -550 4367 50  0000 C CNN
 F 1 "74AHCT04" H -550 4276 50  0000 C CNN
 F 2 "Package_SO:TSSOP-14_4.4x5mm_P0.65mm" H -550 4050 50  0001 C CNN
@@
 AR Path="/5D2C0720/5FC492DE" Ref="U?"  Part="3"
 AR Path="/5D2C07CD/5FC492DE" Ref="U?"  Part="3"
-AR Path="/60A72859/5FC492DE" Ref="U30"  Part="3"
-F 0 "U30" H -550 3867 50  0000 C CNN
+AR Path="/60A72859/5FC492DE" Ref="U29"  Part="3"
+F 0 "U29" H -550 3867 50  0000 C CNN
 F 1 "74AHCT04" H -550 3776 50  0000 C CNN
 F 2 "Package_SO:TSSOP-14_4.4x5mm_P0.65mm" H -550 3550 50  0001 C CNN
@@
 AR Path="/5D2C0720/5FC492E6" Ref="#PWR?"  Part="1"
 AR Path="/5D2C07CD/5FC492E6" Ref="#PWR?"  Part="1"
-AR Path="/60A72859/5FC492E6" Ref="#PWR0127"  Part="1"
-F 0 "#PWR0127" H -850 2000 50  0001 C CNN
+AR Path="/60A72859/5FC492E6" Ref="#PWR0123"  Part="1"
+F 0 "#PWR0123" H -850 2000 50  0001 C CNN
 F 1 "VCC" H -833 2323 50  0000 C CNN
 F 2 "" H -850 2150 50  0001 C CNN
@@
 	1    0    0    -1
 $EndComp
-Wire Wire Line
-	-850 3050 -850 3550
-Connection ~ -850 3050
 Connection ~ -850 3550
 Wire Wire Line
@@
 AR Path="/5D2C0761/5FC492F4" Ref="#PWR?"  Part="1"
 AR Path="/5D2C07CD/5FC492F4" Ref="#PWR?"  Part="1"
-AR Path="/60A72859/5FC492F4" Ref="#PWR0128"  Part="1"
-F 0 "#PWR0128" H -850 6250 50  0001 C CNN
+AR Path="/60A72859/5FC492F4" Ref="#PWR0124"  Part="1"
+F 0 "#PWR0124" H -850 6250 50  0001 C CNN
 F 1 "GND" H -845 6327 50  0000 C CNN
 F 2 "" H -850 6500 50  0001 C CNN
@@
 AR Path="/5D2C0720/5FC492FE" Ref="U?"  Part="2"
 AR Path="/5D2C07CD/5FC492FE" Ref="U?"  Part="1"
-AR Path="/60A72859/5FC492FE" Ref="U30"  Part="1"
-F 0 "U30" H 4650 2467 50  0000 C CNN
+AR Path="/60A72859/5FC492FE" Ref="U29"  Part="1"
+F 0 "U29" H 4650 2467 50  0000 C CNN
 F 1 "74AHCT04" H 4650 2376 50  0000 C CNN
 F 2 "Package_SO:TSSOP-14_4.4x5mm_P0.65mm" H 4650 2150 50  0001 C CNN
@@
 	1    0    0    -1
 $EndComp
-Wire Wire Line
-	-850 2150 -850 3050
 Wire Wire Line
 	4950 2150 5100 2150
@@
 AR Path="/60B264DC/5FCD7CF6/6041A556" Ref="#PWR?"  Part="1"
 AR Path="/60A72859/603C451A/6041A556" Ref="#PWR?"  Part="1"
-AR Path="/60A72859/6041A556" Ref="#PWR0129"  Part="1"
-F 0 "#PWR0129" H 850 6900 50  0001 C CNN
+AR Path="/60A72859/6041A556" Ref="#PWR0125"  Part="1"
+F 0 "#PWR0125" H 850 6900 50  0001 C CNN
 F 1 "VCC" H 867 7223 50  0000 C CNN
 F 2 "" H 850 7050 50  0001 C CNN
@@
 AR Path="/60B264DC/5FCD7CF6/6041A55C" Ref="#PWR?"  Part="1"
 AR Path="/60A72859/603C451A/6041A55C" Ref="#PWR?"  Part="1"
-AR Path="/60A72859/6041A55C" Ref="#PWR0130"  Part="1"
-F 0 "#PWR0130" H 850 7200 50  0001 C CNN
+AR Path="/60A72859/6041A55C" Ref="#PWR0126"  Part="1"
+F 0 "#PWR0126" H 850 7200 50  0001 C CNN
 F 1 "GND" H 855 7277 50  0000 C CNN
 F 2 "" H 850 7450 50  0001 C CNN
@@
 Wire Wire Line
 	5100 3450 5100 4150
+Wire Wire Line
+	-850 2150 -850 3550
 $EndSCHEMATC

Commit message: checkpoint
Parts:
- removed unit 3 of U29
Connections:
- wire segments 18 -> 17
Changed lines of the file:
@@
-	1    0    0    -1
-$EndComp
-$Comp
-L 74xx:74LS04 U?
-U 3 1 5FC492DE
-P -550 3550
-AR Path="/5D8005AF/5D800744/5FC492DE" Ref="U?"  Part="6"
-AR Path="/5D2C0720/5FC492DE" Ref="U?"  Part="3"
-AR Path="/5D2C07CD/5FC492DE" Ref="U?"  Part="3"
-AR Path="/60A72859/5FC492DE" Ref="U29"  Part="3"
-F 0 "U29" H -550 3867 50  0000 C CNN
-F 1 "74AHCT04" H -550 3776 50  0000 C CNN
-F 2 "Package_SO:TSSOP-14_4.4x5mm_P0.65mm" H -550 3550 50  0001 C CNN
-F 3 "http://www.ti.com/general/docs/suppproductinfo.tsp?distId=26&gotoUrl=http%3A%2F%2Fwww.ti.com%2Flit%2Fgpn%2Fsn74ahct04" H -550 3550 50  0001 C CNN
-	3    -550 3550
 	1    0    0    -1
 $EndComp
@@
 	1    0    0    -1
 $EndComp
-Connection ~ -850 3550
-Wire Wire Line
-	-850 3550 -850 4050
 Connection ~ -850 4050
 Wire Wire Line
@@
 	5100 3450 5100 4150
 Wire Wire Line
-	-850 2150 -850 3550
+	-850 2150 -850 4050
 $EndSCHEMATC
