File: RightOperandRegister.sch (KiCad schematic (older format))
At the start: 4 parts, among them U33 74ABT574, U34 74ABT574

Commit message: Update broken footprints for resistors and capacitors.
Parts:
- C34, C35: footprint Capacitor_SMD:C_0603_1608Metric_Pad1.05x0.95mm_HandSolder -> Capacitor_SMD:C_0201_0603Metric_Pad0.64x0.40mm_HandSolder
Changed lines of the file:
@@
 F 0 "C34" H 1415 6996 50  0000 L CNN
 F 1 "100nF" H 1415 6905 50  0000 L CNN
-F 2 "Capacitor_SMD:C_0603_1608Metric_Pad1.05x0.95mm_HandSolder" H 1338 6800 50  0001 C CNN
+F 2 "Capacitor_SMD:C_0201_0603Metric_Pad0.64x0.40mm_HandSolder" H 1338 6800 50  0001 C CNN
 F 3 "~" H 1300 6950 50  0001 C CNN
 	1    1300 6950
@@
 F 0 "C35" H 1865 6996 50  0000 L CNN
 F 1 "100nF" H 1865 6905 50  0000 L CNN
-F 2 "Capacitor_SMD:C_0603_1608Metric_Pad1.05x0.95mm_HandSolder" H 1788 6800 50  0001 C CNN
+F 2 "Capacitor_SMD:C_0201_0603Metric_Pad0.64x0.40mm_HandSolder" H 1788 6800 50  0001 C CNN
 F 3 "~" H 1750 6950 50  0001 C CNN
 	1    1750 6950

Commit message: Fix typo in ID
Parts:
- C34, C35: footprint Capacitor_SMD:C_0201_0603Metric_Pad0.64x0.40mm_HandSolder -> Capacitor_SMD:C_0603_1608Metric_Pad1.08x0.95mm_HandSolder
Changed lines of the file:
@@
 F 0 "C34" H 1415 6996 50  0000 L CNN
 F 1 "100nF" H 1415 6905 50  0000 L CNN
-F 2 "Capacitor_SMD:C_0201_0603Metric_Pad0.64x0.40mm_HandSolder" H 1338 6800 50  0001 C CNN
+F 2 "Capacitor_SMD:C_0603_1608Metric_Pad1.08x0.95mm_HandSolder" H 1338 6800 50  0001 C CNN
 F 3 "~" H 1300 6950 50  0001 C CNN
 	1    1300 6950
@@
 F 0 "C35" H 1865 6996 50  0000 L CNN
 F 1 "100nF" H 1865 6905 50  0000 L CNN
-F 2 "Capacitor_SMD:C_0201_0603Metric_Pad0.64x0.40mm_HandSolder" H 1788 6800 50  0001 C CNN
+F 2 "Capacitor_SMD:C_0603_1608Metric_Pad1.08x0.95mm_HandSolder" H 1788 6800 50  0001 C CNN
 F 3 "~" H 1750 6950 50  0001 C CNN
 	1    1750 6950

Commit message: Checkpoint while routing PCB.
A lot of parts have been placed and about a quarter of the board is routed.
Parts:
- renumbered U33 to U32, U34 to U33
Changed lines of the file:
@@
 AR Path="/60B264DC/5FCD7CF6/603E19AC" Ref="#PWR?"  Part="1"
 AR Path="/60A8EF0C/604A048B/603E19AC" Ref="#PWR?"  Part="1"
-AR Path="/60A72859/603DC723/603E19AC" Ref="#PWR0145"  Part="1"
-F 0 "#PWR0145" H 5350 2650 50  0001 C CNN
+AR Path="/60A72859/603DC723/603E19AC" Ref="#PWR0141"  Part="1"
+F 0 "#PWR0141" H 5350 2650 50  0001 C CNN
 F 1 "GND" V 5355 2772 50  0000 R CNN
 F 2 "" H 5350 2900 50  0001 C CNN
@@
 AR Path="/60B264DC/5FCD7CF6/603E19CC" Ref="#PWR?"  Part="1"
 AR Path="/60A8EF0C/604A048B/603E19CC" Ref="#PWR?"  Part="1"
-AR Path="/60A72859/603DC723/603E19CC" Ref="#PWR0148"  Part="1"
-F 0 "#PWR0148" H 5850 2950 50  0001 C CNN
+AR Path="/60A72859/603DC723/603E19CC" Ref="#PWR0144"  Part="1"
+F 0 "#PWR0144" H 5850 2950 50  0001 C CNN
 F 1 "GND" H 5855 3027 50  0000 C CNN
 F 2 "" H 5850 3200 50  0001 C CNN
@@
 AR Path="/60B264DC/5FCD7CF6/603E19D2" Ref="#PWR?"  Part="1"
 AR Path="/60A8EF0C/604A048B/603E19D2" Ref="#PWR?"  Part="1"
-AR Path="/60A72859/603DC723/603E19D2" Ref="#PWR0147"  Part="1"
-F 0 "#PWR0147" H 5850 1450 50  0001 C CNN
+AR Path="/60A72859/603DC723/603E19D2" Ref="#PWR0143"  Part="1"
+F 0 "#PWR0143" H 5850 1450 50  0001 C CNN
 F 1 "VCC" H 5867 1773 50  0000 C CNN
 F 2 "" H 5850 1600 50  0001 C CNN
@@
 AR Path="/60B264DC/5FCD7CF6/603E19F2" Ref="U?"  Part="1"
 AR Path="/60A8EF0C/604A048B/603E19F2" Ref="U?"  Part="1"
-AR Path="/60A72859/603DC723/603E19F2" Ref="U33"  Part="1"
-F 0 "U33" H 5600 3200 50  0000 C CNN
+AR Path="/60A72859/603DC723/603E19F2" Ref="U32"  Part="1"
+F 0 "U32" H 5600 3200 50  0000 C CNN
 F 1 "74ABT574" H 5600 3100 50  0000 C CNN
 F 2 "Package_SO:TSSOP-20_4.4x6.5mm_P0.65mm" H 5850 2400 50  0001 C CNN
@@
 AR Path="/60B264DC/5FCD7CF6/603E19FE" Ref="#PWR?"  Part="1"
 AR Path="/60A8EF0C/604A048B/603E19FE" Ref="#PWR?"  Part="1"
-AR Path="/60A72859/603DC723/603E19FE" Ref="#PWR0141"  Part="1"
-F 0 "#PWR0141" H 1300 6650 50  0001 C CNN
+AR Path="/60A72859/603DC723/603E19FE" Ref="#PWR0137"  Part="1"
+F 0 "#PWR0137" H 1300 6650 50  0001 C CNN
 F 1 "VCC" H 1317 6973 50  0000 C CNN
 F 2 "" H 1300 6800 50  0001 C CNN
@@
 AR Path="/60B264DC/5FCD7CF6/603E1A04" Ref="#PWR?"  Part="1"
 AR Path="/60A8EF0C/604A048B/603E1A04" Ref="#PWR?"  Part="1"
-AR Path="/60A72859/603DC723/603E1A04" Ref="#PWR0142"  Part="1"
-F 0 "#PWR0142" H 1300 6950 50  0001 C CNN
+AR Path="/60A72859/603DC723/603E1A04" Ref="#PWR0138"  Part="1"
+F 0 "#PWR0138" H 1300 6950 50  0001 C CNN
 F 1 "GND" H 1305 7027 50  0000 C CNN
 F 2 "" H 1300 7200 50  0001 C CNN
@@
 AR Path="/60B264DC/5FCD7CF6/603E1A11" Ref="#PWR?"  Part="1"
 AR Path="/60A8EF0C/604A048B/603E1A11" Ref="#PWR?"  Part="1"
-AR Path="/60A72859/603DC723/603E1A11" Ref="#PWR0143"  Part="1"
-F 0 "#PWR0143" H 1750 6650 50  0001 C CNN
+AR Path="/60A72859/603DC723/603E1A11" Ref="#PWR0139"  Part="1"
+F 0 "#PWR0139" H 1750 6650 50  0001 C CNN
 F 1 "VCC" H 1767 6973 50  0000 C CNN
 F 2 "" H 1750 6800 50  0001 C CNN
@@
 AR Path="/60B264DC/5FCD7CF6/603E1A17" Ref="#PWR?"  Part="1"
 AR Path="/60A8EF0C/604A048B/603E1A17" Ref="#PWR?"  Part="1"
-AR Path="/60A72859/603DC723/603E1A17" Ref="#PWR0144"  Part="1"
-F 0 "#PWR0144" H 1750 6950 50  0001 C CNN
+AR Path="/60A72859/603DC723/603E1A17" Ref="#PWR0140"  Part="1"
+F 0 "#PWR0140" H 1750 6950 50  0001 C CNN
 F 1 "GND" H 1755 7027 50  0000 C CNN
 F 2 "" H 1750 7200 50  0001 C CNN
@@
 AR Path="/60B264DC/5FCD7CF6/603E1A1F" Ref="#PWR?"  Part="1"
 AR Path="/60A8EF0C/604A048B/603E1A1F" Ref="#PWR?"  Part="1"
-AR Path="/60A72859/603DC723/603E1A1F" Ref="#PWR0146"  Part="1"
-F 0 "#PWR0146" H 5350 4700 50  0001 C CNN
+AR Path="/60A72859/603DC723/603E1A1F" Ref="#PWR0142"  Part="1"
+F 0 "#PWR0142" H 5350 4700 50  0001 C CNN
 F 1 "GND" V 5355 4822 50  0000 R CNN
 F 2 "" H 5350 4950 50  0001 C CNN
@@
 AR Path="/60B264DC/5FCD7CF6/603E1A3E" Ref="#PWR?"  Part="1"
 AR Path="/60A8EF0C/604A048B/603E1A3E" Ref="#PWR?"  Part="1"
-AR Path="/60A72859/603DC723/603E1A3E" Ref="#PWR0150"  Part="1"
-F 0 "#PWR0150" H 5850 5000 50  0001 C CNN
+AR Path="/60A72859/603DC723/603E1A3E" Ref="#PWR0146"  Part="1"
+F 0 "#PWR0146" H 5850 5000 50  0001 C CNN
 F 1 "GND" H 5855 5077 50  0000 C CNN
 F 2 "" H 5850 5250 50  0001 C CNN
@@
 AR Path="/60B264DC/5FCD7CF6/603E1A44" Ref="#PWR?"  Part="1"
 AR Path="/60A8EF0C/604A048B/603E1A44" Ref="#PWR?"  Part="1"
-AR Path="/60A72859/603DC723/603E1A44" Ref="#PWR0149"  Part="1"
-F 0 "#PWR0149" H 5850 3500 50  0001 C CNN
+AR Path="/60A72859/603DC723/603E1A44" Ref="#PWR0145"  Part="1"
+F 0 "#PWR0145" H 5850 3500 50  0001 C CNN
 F 1 "VCC" H 5867 3823 50  0000 C CNN
 F 2 "" H 5850 3650 50  0001 C CNN
@@
 AR Path="/60B264DC/5FCD7CF6/603E1A62" Ref="U?"  Part="1"
 AR Path="/60A8EF0C/604A048B/603E1A62" Ref="U?"  Part="1"
-AR Path="/60A72859/603DC723/603E1A62" Ref="U34"  Part="1"
-F 0 "U34" H 5600 5250 50  0000 C CNN
+AR Path="/60A72859/603DC723/603E1A62" Ref="U33"  Part="1"
+F 0 "U33" H 5600 5250 50  0000 C CNN
 F 1 "74ABT574" H 5600 5150 50  0000 C CNN
 F 2 "Package_SO:TSSOP-20_4.4x6.5mm_P0.65mm" H 5850 4450 50  0001 C CNN
