File: Backplane/BypassPrototypeInputs.kicad_sch (KiCad schematic)
At the start: 5 parts, among them J36 RegisterA, J37 RegisterB, J38 Y_MEM, J39 Y_EX, J40 Control Signals

Commit message: Backplane: Fix several unconnected signals
Several signals and control lines were not connected on the backplane PCB
in Rev A and these are all fixed now.

Also, update to KiCad 7
Parts:
- J36, J37, J38, J39: symbol Connector:Conn_01x16_Male -> Connector:Conn_01x16_Pin
- J40: symbol Connector:Conn_01x10_Male -> Connector:Conn_01x10_Pin
