File: Backplane/EXPrototypeOutputs.kicad_sch (KiCad schematic)
At the start: 8 parts, among them J48 StoreOp_MEM, J49 Y_EX, J50 Y_MEM, J51 Y_EX, J52 Y_MEM, J53 Flags, J54 SelC_MEM, J55 Y_EX

Commit message: Backplane: Fix several unconnected signals
Several signals and control lines were not connected on the backplane PCB
in Rev A and these are all fixed now.

Also, update to KiCad 7
Parts:
- J48, J49, J50, J51, J52: symbol Connector:Conn_01x16_Male -> Connector:Conn_01x16_Pin
- J53: symbol Connector:Conn_01x04_Male -> Connector:Conn_01x04_Pin
- J54: symbol Connector:Conn_01x03_Male -> Connector:Conn_01x03_Pin
- J55: symbol Connector:Conn_01x07_Male -> Connector:Conn_01x07_Pin
