File: MEMModule-NoROM/MEM.kicad_sch (KiCad schematic)
At the start: 5 parts, among them U1 74ABT32, U2 74AHCT04

Commit message: MEMModule: Fix bug in the bank register reset signal
The bank register expects an active-high reset signal but was wired to
receive an active-low signal. Fix this issue by routing /RST_sync through
an inverter first.

BUG: The MainBoard PCB layout has not been updated yet.
Parts:
- removed unit 6 of U2
Connections:
- no-connect marks 6 -> 5
Changed lines of the file:
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@@
   (junction (at -21.59 120.65) (diameter 0) (color 0 0 0 0)
   )
-  (junction (at -21.59 146.05) (diameter 0) (color 0 0 0 0)
-  )
   (junction (at -44.45 140.97) (diameter 0) (color 0 0 0 0)
   )
@@
   (junction (at 27.94 182.88) (diameter 0) (color 0 0 0 0)
   )
-  (no_connect (at -6.35 146.05))
   (no_connect (at -6.35 107.95))
   (no_connect (at -26.67 128.27))
@@
     (stroke (width 0) (type default))
   )
-  (wire (pts (xy -21.59 133.35) (xy -21.59 146.05))
+  (wire (pts (xy -21.59 133.35) (xy -21.59 153.67))
     (stroke (width 0) (type default))
   )
@@
   )
   (wire (pts (xy -44.45 140.97) (xy -44.45 146.05))
-    (stroke (width 0) (type default))
-  )
-  (wire (pts (xy -21.59 146.05) (xy -21.59 153.67))
     (stroke (width 0) (type default))
   )
@@
         )
       )
-    )
-  )
-  (symbol (lib_id "74xx:74LS04") (at -13.97 146.05 0) (unit 6)
-    (in_bom yes) (on_board yes) (dnp no)
-    (property "Reference" "U2" (at -13.97 137.9982 0)
-      (effects (font (size 1.27 1.27)))
-    )
-    (property "Value" "74AHCT04" (at -13.97 140.3096 0)
-      (effects (font (size 1.27 1.27)))
-    )
-    (property "Footprint" "Package_SO:TSSOP-14_4.4x5mm_P0.65mm" (at -13.97 146.05 0)
-      (effects (font (size 1.27 1.27)) hide)
-    )
-    (property "Datasheet" "http://www.ti.com/lit/gpn/sn74LS04" (at -13.97 146.05 0)
-      (effects (font (size 1.27 1.27)) hide)
-    )
-    (property "Mouser" "https://www.mouser.com/ProductDetail/771-AHCT04PW112" (at -13.97 146.05 0)
-      (effects (font (size 1.27 1.27)) hide)
-    )
-    (pin "1")
-    (pin "2")
-    (pin "3")
-    (pin "4")
-    (pin "5")
-    (pin "6")
-    (pin "8")
-    (pin "9")
-    (pin "10")
-    (pin "11")
-    (pin "12")
-    (pin "13")
-    (pin "14")
-    (pin "7")
-    (instances
-      (project "MEMModule"
-        (path "/83c5181e-f5ee-453c-ae5c-d7256ba8837d/00000000-0000-0000-0000-000060af64de"
-          (reference "U2") (unit 6)
-        )
-      )
