File: ProcessorBoard/Program Counter.kicad_sch (KiCad schematic)
At the start: 8 parts, among them U57 74ABT32, U58 74AHCT04, U59 IDT7381

Commit message: ProcessorBoard: update to include M/S bug fix in register file
Parts:
- renumbered C62 to C56, C63 to C57, C64 to C58, TP75 to TP68, TP76 to TP69, U57 to U53, U58 to U54, U59 to U55

Commit message: ProcessorBoard: Replace Instruction ROM with a header for a daughter board
ROMs will be relocated to a daughter board to allow the memories and their
sockets to be swapped easily.
Parts:
- renumbered C56 to C54, C57 to C55, C58 to C56, TP68 to TP62, TP69 to TP63, U53 to U51, U54 to U52, U55 to U53

Commit message: ProcessorBoard: Copy symbols into project symbol library, make consistent
Symbols created for Turtle16 have been copied into a project-specific
symbol library. The symbols have all been updated with manufacturer,
manufacturer part number, mouser part number, and digikey part number.

Test points and mounting holes have been marked to be excluded from BOM.
Parts:
- C54, C55, C56: footprint Capacitor_SMD:C_0603_1608Metric_Pad1.08x0.95mm_HandSolder -> Capacitor_SMD:C_0603_1608Metric; Digikey# (none) -> 587-6004-1-ND; Manufacturer (none) -> Taiyo Yuden; Manufacturer# (none) -> EMK107B7104KAHT; Mouser https://www.mouser.com/ProductDetail/963-EMK107B7104KAHT -> (none); Mouser# (none) -> 963-EMK107B7104KAHT
- TP62, TP63: now left out of the parts list
- U51: symbol 74xx:74LS32 -> Turtle16:74ABT32; Digikey# (none) -> 1727-6509-1-ND; Manufacturer (none) -> Nexperia; Manufacturer# (none) -> 74ABT32PW,118; Mouser https://www.mouser.com/ProductDetail/Nexperia/74ABT32PW118?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 -> (none); Mouser# (none) -> 771-ABT32PW118
- U52: symbol 74xx:74LS04 -> Turtle16:74AHCT04; Digikey# (none) -> 1727-74AHCT04APWJCT-ND; Manufacturer (none) -> Nexperia; Manufacturer# (none) -> 74AHCT04APWJ; Mouser https://www.mouser.com/ProductDetail/771-AHCT04PW112 -> (none); Mouser# (none) -> 771-74AHCT04APWJ
- U53: symbol PCIFModule-rescue:IDT7381-CPU -> Turtle16:IDT7381; Digikey# (none) -> 3M6821B1-ND; Manufacturer (none) -> 3M; Manufacturer# (none) -> 8468-21B1-RK-TP; Mouser https://www.mouser.com/ProductDetail/3M-Electronic-Solution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 -> (none); Mouser# (none) -> 517-8468-21B1-RK-TP
