File: Hardware/MonolithicProcessor/ProcessorBoardTestFixture/LEDOutputs.kicad_sch (KiCad schematic)
At the start: 18 parts, among them U11 74HC595

Commit message: Update all KiCAD projects to KiCAD 9
Parts:
- renumbered U11 to U10
