File: Hardware/PrototypeProcessor/MEMModule/ROM.kicad_sch (KiCad schematic)
At the start: 4 parts, among them U11 SST39SF010

Commit message: Update all KiCAD projects to KiCAD 9
Parts:
- renumbered C10 to C14, C11 to C15, U11 to U12
