File: Hardware/CardProcessor/MainBoard/HazardControlComparators.kicad_sch (KiCad schematic)
At the start: 12 parts, among them U16 74F521, U17 74F521, U18 74F521, U19 74F521

Commit message: Extract ID to new ControlModule sheet
Parts:
- renumbered C17 to C78, C18 to C79, C19 to C80, C20 to C81, TP31 to TP133, TP32 to TP134, TP33 to TP135, TP34 to TP136, U16 to U75, U17 to U76, U18 to U77, U19 to U78

Commit message: Reannotate schematic by hand since extracting to new sheets broke existing annotations
Parts:
- renumbered C78 to C17, C79 to C18, C80 to C19, C81 to C20, TP133 to TP31, TP134 to TP32, TP135 to TP33, TP136 to TP34, U75 to U16, U76 to U17, U77 to U18, U78 to U19
Changed lines of the file:
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@@
 		(on_board yes)
 		(dnp no)
-		(property "Reference" "C78"
+		(property "Reference" "C17"
 			(at 21.971 188.0616 0)
 			(effects
@@
 			(project "MainBoard"
 				(path "/83c5181e-f5ee-453c-ae5c-d7256ba8837d/333b4292-93f5-442d-a859-8b1da2cd4698/101aadd6-c8f8-4873-8d28-86528ab686cf/00000000-0000-0000-0000-00005fda967f/00000000-0000-0000-0000-0000606fef6b"
-					(reference "C78")
+					(reference "C17")
 					(unit 1)
 				)
@@
 		(on_board yes)
 		(dnp no)
-		(property "Reference" "C79"
+		(property "Reference" "C18"
 			(at 34.671 188.0616 0)
 			(effects
@@
 			(project "MainBoard"
 				(path "/83c5181e-f5ee-453c-ae5c-d7256ba8837d/333b4292-93f5-442d-a859-8b1da2cd4698/101aadd6-c8f8-4873-8d28-86528ab686cf/00000000-0000-0000-0000-00005fda967f/00000000-0000-0000-0000-0000606fef6b"
-					(reference "C79")
+					(reference "C18")
 					(unit 1)
 				)
@@
 		(on_board yes)
 		(dnp no)
-		(property "Reference" "C80"
+		(property "Reference" "C19"
 			(at 47.371 188.0616 0)
 			(effects
@@
 			(project "MainBoard"
 				(path "/83c5181e-f5ee-453c-ae5c-d7256ba8837d/333b4292-93f5-442d-a859-8b1da2cd4698/101aadd6-c8f8-4873-8d28-86528ab686cf/00000000-0000-0000-0000-00005fda967f/00000000-0000-0000-0000-0000606fef6b"
-					(reference "C80")
+					(reference "C19")
 					(unit 1)
 				)
@@
 		(on_board yes)
 		(dnp no)
-		(property "Reference" "C81"
+		(property "Reference" "C20"
 			(at 60.071 188.0616 0)
 			(effects
@@
 			(project "MainBoard"
 				(path "/83c5181e-f5ee-453c-ae5c-d7256ba8837d/333b4292-93f5-442d-a859-8b1da2cd4698/101aadd6-c8f8-4873-8d28-86528ab686cf/00000000-0000-0000-0000-00005fda967f/00000000-0000-0000-0000-0000606fef6b"
-					(reference "C81")
+					(reference "C20")
 					(unit 1)
 				)
@@
 		(on_board yes)
 		(dnp no)
-		(property "Reference" "U75"
+		(property "Reference" "U16"
 			(at 102.87 66.04 0)
 			(effects
@@
 			(project "MainBoard"
 				(path "/83c5181e-f5ee-453c-ae5c-d7256ba8837d/333b4292-93f5-442d-a859-8b1da2cd4698/101aadd6-c8f8-4873-8d28-86528ab686cf/00000000-0000-0000-0000-00005fda967f/00000000-0000-0000-0000-0000606fef6b"
-					(reference "U75")
+					(reference "U16")
 					(unit 1)
 				)
@@
 		(on_board yes)
 		(dnp no)
-		(property "Reference" "U76"
+		(property "Reference" "U17"
 			(at 102.87 128.27 0)
 			(effects
@@
 			(project "MainBoard"
 				(path "/83c5181e-f5ee-453c-ae5c-d7256ba8837d/333b4292-93f5-442d-a859-8b1da2cd4698/101aadd6-c8f8-4873-8d28-86528ab686cf/00000000-0000-0000-0000-00005fda967f/00000000-0000-0000-0000-0000606fef6b"
-					(reference "U76")
+					(reference "U17")
 					(unit 1)
 				)
@@
 		(on_board yes)
 		(dnp no)
-		(property "Reference" "U78"
+		(property "Reference" "U19"
 			(at 234.95 66.04 0)
 			(effects
@@
 			(project "MainBoard"
 				(path "/83c5181e-f5ee-453c-ae5c-d7256ba8837d/333b4292-93f5-442d-a859-8b1da2cd4698/101aadd6-c8f8-4873-8d28-86528ab686cf/00000000-0000-0000-0000-00005fda967f/00000000-0000-0000-0000-0000606fef6b"
-					(reference "U78")
+					(reference "U19")
 					(unit 1)
 				)
@@
 		(on_board yes)
 		(dnp no)
-		(property "Reference" "U77"
+		(property "Reference" "U18"
 			(at 218.44 121.92 0)
 			(effects
@@
 			(project "MainBoard"
 				(path "/83c5181e-f5ee-453c-ae5c-d7256ba8837d/333b4292-93f5-442d-a859-8b1da2cd4698/101aadd6-c8f8-4873-8d28-86528ab686cf/00000000-0000-0000-0000-00005fda967f/00000000-0000-0000-0000-0000606fef6b"
-					(reference "U77")
+					(reference "U18")
 					(unit 1)
 				)
@@
 		(on_board yes)
 		(dnp no)
-		(fields_autoplaced yes)
-		(property "Reference" "TP136"
-			(at 218.567 24.765 90)
-			(effects
-				(font
-					(size 1.27 1.27)
-				)
+		(property "Reference" "TP34"
+			(at 220.98 31.496 90)
+			(effects
+				(font
+					(size 1.27 1.27)
+				)
+				(justify left)
 			)
 		)
 		(property "Value" "SEL_B_MATCHES_SEL_C_EX"
-			(at 218.567 27.305 90)
-			(effects
-				(font
-					(size 1.27 1.27)
-				)
+			(at 220.98 33.274 90)
+			(effects
+				(font
+					(size 1.27 1.27)
+				)
+				(justify left)
 			)
 		)
@@
 			(project "MainBoard"
 				(path "/83c5181e-f5ee-453c-ae5c-d7256ba8837d/333b4292-93f5-442d-a859-8b1da2cd4698/101aadd6-c8f8-4873-8d28-86528ab686cf/00000000-0000-0000-0000-00005fda967f/00000000-0000-0000-0000-0000606fef6b"
-					(reference "TP136")
+					(reference "TP34")
 					(unit 1)
 				)
@@
 		(on_board yes)
 		(dnp no)
-		(fields_autoplaced yes)
-		(property "Reference" "TP133"
-			(at 167.767 15.24 90)
-			(effects
-				(font
-					(size 1.27 1.27)
-				)
+		(property "Reference" "TP31"
+			(at 166.878 17.018 90)
+			(effects
+				(font
+					(size 1.27 1.27)
+				)
+				(justify left)
 			)
 		)
 		(property "Value" "SEL_B_MATCHES_SEL_C_MEM"
-			(at 167.767 17.78 90)
-			(effects
-				(font
-					(size 1.27 1.27)
-				)
+			(at 166.878 19.05 90)
+			(effects
+				(font
+					(size 1.27 1.27)
+				)
+				(justify left)
 			)
 		)
@@
 			(project "MainBoard"
 				(path "/83c5181e-f5ee-453c-ae5c-d7256ba8837d/333b4292-93f5-442d-a859-8b1da2cd4698/101aadd6-c8f8-4873-8d28-86528ab686cf/00000000-0000-0000-0000-00005fda967f/00000000-0000-0000-0000-0000606fef6b"
-					(reference "TP133")
+					(reference "TP31")
 					(unit 1)
 				)
@@
 		(on_board yes)
 		(dnp no)
-		(property "Reference" "TP135"
-			(at 202.057 22.225 90)
+		(property "Reference" "TP33"
+			(at 205.74 26.162 90)
 			(effects
 				(font
@@
 		)
 		(property "Value" "SEL_A_MATCHES_SEL_C_EX"
-			(at 202.057 24.765 90)
+			(at 215.9 27.94 90)
 			(effects
 				(font
@@
 			(project "MainBoard"
 				(path "/83c5181e-f5ee-453c-ae5c-d7256ba8837d/333b4292-93f5-442d-a859-8b1da2cd4698/101aadd6-c8f8-4873-8d28-86528ab686cf/00000000-0000-0000-0000-00005fda967f/00000000-0000-0000-0000-0000606fef6b"
-					(reference "TP135")
+					(reference "TP33")
 					(unit 1)
 				)
@@
 		(on_board yes)
 		(dnp no)
-		(fields_autoplaced yes)
-		(property "Reference" "TP134"
-			(at 184.912 19.05 90)
-			(effects
-				(font
-					(size 1.27 1.27)
-				)
+		(property "Reference" "TP32"
+			(at 183.388 21.082 90)
+			(effects
+				(font
+					(size 1.27 1.27)
+				)
+				(justify left)
 			)
 		)
 		(property "Value" "SEL_A_MATCHES_SEL_C_MEM"
-			(at 184.912 21.59 90)
-			(effects
-				(font
-					(size 1.27 1.27)
-				)
+			(at 183.388 22.86 90)
+			(effects
+				(font
+					(size 1.27 1.27)
+				)
+				(justify left)
 			)
 		)
@@
 			(project "MainBoard"
 				(path "/83c5181e-f5ee-453c-ae5c-d7256ba8837d/333b4292-93f5-442d-a859-8b1da2cd4698/101aadd6-c8f8-4873-8d28-86528ab686cf/00000000-0000-0000-0000-00005fda967f/00000000-0000-0000-0000-0000606fef6b"
-					(reference "TP134")
-					(unit 1)
-				)
+					(reference "TP32")
+					(unit 1)
+				)

Commit message: Automatically reannotate project and fix a few silkscreen-related issues
Parts:
- renumbered C17 to C36, C18 to C37, C19 to C38, C20 to C39, TP31 to TP60, TP32 to TP61, TP33 to TP62, TP34 to TP63, U16 to U33, U17 to U34, U18 to U35, U19 to U36
