File: Hardware/CardProcessor/RegisterFileCard/SelectWriteBackSource.kicad_sch (KiCad schematic)
At the start: 8 parts, among them U1 74AHCT138, U2 74ABT16245, U3 74ABT16245

Commit message: Annotate schematics such that Turtle16Computer can perform ERC and DRC
- Turtle16Computer must be fully annotated to perform ERC on the schematic.
Also, the PCB cannot be updated without full annotations either. However,
KiCad projects for individual PCBs must also remain annotated and capable
of updating the PCB and performing ERC and DRC.

- Manually set KiCad project fields to "" in kicad_sch files

- Manually replace the UUID of EXCard so it no longer collides with the
UUI of the Turtle16Computer project.
Parts:
- renumbered C3 to C10, C1 to C8, C2 to C9, TP17 to TP4, TP18 to TP5, U2 to U6, U3 to U7, U1 to U8

Commit message: Ensure all cards have a unique 4-bit identifier code and proper power pins
The pinout on all cards will devote the first four pins to the identifier,
followed by four pins for +5V, and four pins for GND. This allows a card to
draw up to about 2 amps.
Parts:
- renumbered C8 to C1, C9 to C2, C10 to C3, TP4 to TP17, TP5 to TP18, U8 to U1, U6 to U2, U7 to U3
Changed lines of the file:
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@@
 		(on_board yes)
 		(dnp no)
-		(property "Reference" "#PWR0437"
+		(property "Reference" "#PWR09"
 			(at 80.01 88.9 0)
 			(effects
@@
 		(on_board yes)
 		(dnp no)
-		(property "Reference" "#PWR0442"
+		(property "Reference" "#PWR01"
 			(at 34.29 161.29 0)
 			(effects
@@
 		(on_board yes)
 		(dnp no)
-		(property "Reference" "C8"
+		(property "Reference" "C1"
 			(at 77.851 189.3316 0)
 			(effects
@@
 		(on_board yes)
 		(dnp no)
-		(property "Reference" "C9"
+		(property "Reference" "C2"
 			(at 90.551 189.3316 0)
 			(effects
@@
 		(on_board yes)
 		(dnp no)
-		(property "Reference" "#PWR0447"
+		(property "Reference" "#PWR07"
 			(at 74.93 190.5 0)
 			(effects
@@
 		(on_board yes)
 		(dnp no)
-		(property "Reference" "#PWR0448"
+		(property "Reference" "#PWR08"
 			(at 74.93 203.2 0)
 			(effects
@@
 		(on_board yes)
 		(dnp no)
-		(property "Reference" "C10"
+		(property "Reference" "C3"
 			(at 101.981 189.3316 0)
 			(effects
@@
 		(on_board yes)
 		(dnp no)
-		(property "Reference" "#PWR0446"
+		(property "Reference" "#PWR06"
 			(at 55.88 193.04 0)
 			(effects
@@
 		(on_board yes)
 		(dnp no)
-		(property "Reference" "#PWR0441"
+		(property "Reference" "#PWR05"
 			(at 55.88 153.67 0)
 			(effects
@@
 		(on_board yes)
 		(dnp no)
-		(property "Reference" "#PWR0443"
+		(property "Reference" "#PWR02"
 			(at 34.29 163.83 0)
 			(effects
@@
 		(on_board yes)
 		(dnp no)
-		(property "Reference" "#PWR0445"
+		(property "Reference" "#PWR04"
 			(at 34.29 175.26 0)
 			(effects
@@
 		(on_board yes)
 		(dnp no)
-		(property "Reference" "#PWR0444"
+		(property "Reference" "#PWR03"
 			(at 44.45 171.45 0)
 			(effects
@@
 		(on_board yes)
 		(dnp no)
-		(property "Reference" "#PWR0439"
+		(property "Reference" "#PWR011"
 			(at 104.14 109.22 0)
 			(effects
@@
 		(on_board yes)
 		(dnp no)
-		(property "Reference" "#PWR0435"
+		(property "Reference" "#PWR010"
 			(at 92.71 41.91 0)
 			(effects
@@
 		(on_board yes)
 		(dnp no)
-		(property "Reference" "U6"
+		(property "Reference" "U2"
 			(at 92.71 68.58 0)
 			(effects
@@
 		(on_board yes)
 		(dnp no)
-		(property "Reference" "#PWR0438"
+		(property "Reference" "#PWR012"
 			(at 162.56 88.9 0)
 			(effects
@@
 		(on_board yes)
 		(dnp no)
-		(property "Reference" "#PWR0440"
+		(property "Reference" "#PWR014"
 			(at 186.69 109.22 0)
 			(effects
@@
 		(on_board yes)
 		(dnp no)
-		(property "Reference" "#PWR0436"
+		(property "Reference" "#PWR013"
 			(at 175.26 41.91 0)
 			(effects
@@
 		(on_board yes)
 		(dnp no)
-		(property "Reference" "U7"
+		(property "Reference" "U3"
 			(at 175.26 68.58 0)
 			(effects
@@
 		(on_board yes)
 		(dnp no)
-		(property "Reference" "U8"
+		(property "Reference" "U1"
 			(at 48.26 151.13 0)
 			(effects
@@
 		(on_board yes)
 		(dnp no)
-		(property "Reference" "TP4"
+		(property "Reference" "TP17"
 			(at 78.74 156.21 90)
 			(effects
@@
 		(on_board yes)
 		(dnp no)
-		(property "Reference" "TP5"
+		(property "Reference" "TP18"
 			(at 161.29 158.75 90)
 			(effects
